File: CPUMCU_experiment_interface.sch (KiCad schematic (older format))
At the start: 4 parts, among them J1 LCD Connector, U1 6581SID

Commit message: Added EPROM and temporary microSD card reader
microSD card reader will probably be replaced.
Parts:
- added J1: Micro_SD_Card_Det_Hirose_DM3AT, microSD:microSD_HC_Hirose_DM3D-SF, symbol Connector:Micro_SD_Card_Det_Hirose_DM3AT
- added U2: 27C256, Package_DIP:DIP-28_W15.24mm, symbol Memory_EPROM:27C256
- renumbered J1 to J2
Connections:
- net labels added: A10, A11, A12, A13, A14, A5, A6, A7, A8, A9, LCD_E, LCD_RS, SID_CLK, ~EPROM_OE, ~SID_CS, ~SID_RES
- wire segments 40 -> 76

Commit message: Added 8 SPST switches
Added 8 SPST switches and an 8-resistor array.
Parts:
- added RN?: R_Network08, Resistor_THT:R_Array_SIP9, symbol Device:R_Network08
- added SW? (x8): SW_Push, symbol Switch:SW_Push
Connections:
- net labels added: GNDD
- wire segments 76 -> 105
